File: hardware/v1.0.0/RPi_ADC_hat.sch (EAGLE design)
At the start: 61 parts, among them Q1 FDT439N, Q2 FDT439N, U1 MCP1790, U2 NME0509SC, U3 HIH6131, U4 MCP3424, U5 PCA9517A, U6 LM61 *, U7 C24C32, X1 I2C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

Commit message: Increase gate resistors, renumber parts
Resistors on FET gate increased to more closely match the value
that would be needed if the FET is replaced by a BJT.
Parts:
- JP1: value I2C ADDRESS -> I2C VIN; device pinhead:PINHD-2X3 -> SparkFun:JUMPER-3PTH
- JP2: value PROG -> I2C ADDRESS; device SparkFun:JUMPER-2PTH -> pinhead:PINHD-2X3
- JP3: value I2C VIN -> PROG; device SparkFun:JUMPER-3PTH -> SparkFun:JUMPER-2PTH
- R10, R11: value 330R -> 560R
Connections:
- net 5V_PI: now also JP1.1; no longer JP3.1
- net AVCC: now also JP2.1, JP2.2; no longer JP1.1, JP1.2
- net DC-DC_OUT: now also JP1.3; no longer JP3.3
- net EEPROM_WP: now also JP3.1; no longer JP2.1
- net GND: now also JP2.5, JP2.6, JP3.2; no longer JP1.5, JP1.6, JP2.2
- net I2C_VIN: now also JP1.2; no longer JP3.2
- net N$16: now also JP2.4; no longer JP1.4
- net N$6: now also JP2.3; no longer JP1.3
Changed lines of the file:
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@@
 <part name="GND1" library="supply1" deviceset="GND" device=""/>
 <part name="R12" library="SteveMarple" deviceset="RESISTOR" device="1206-HAND" value="1M"/>
-<part name="R10" library="SteveMarple" deviceset="RESISTOR" device="1206-HAND" value="330R"/>
+<part name="R10" library="SteveMarple" deviceset="RESISTOR" device="1206-HAND" value="560R"/>
 <part name="GND47" library="supply1" deviceset="GND" device=""/>
 <part name="D1" library="SteveMarple" deviceset="DIODE" device="SOT23-1-3-HAND" value="BAS21"/>
@@
 <part name="C19" library="SteveMarple" deviceset="C-EU" device="1206-HAND" value="1u"/>
 <part name="R13" library="SteveMarple" deviceset="RESISTOR" device="1206-HAND" value="1M"/>
-<part name="R11" library="SteveMarple" deviceset="RESISTOR" device="1206-HAND" value="330R"/>
+<part name="R11" library="SteveMarple" deviceset="RESISTOR" device="1206-HAND" value="560R"/>
 <part name="GND5" library="supply1" deviceset="GND" device=""/>
 <part name="D2" library="SteveMarple" deviceset="DIODE" device="SOT23-1-3-HAND" value="BAS21"/>
@@
 <part name="C12" library="SteveMarple" deviceset="C-EU" device="1206-HAND" value="100p"/>
 <part name="C13" library="SteveMarple" deviceset="C-EU" device="1206-HAND" value="100p"/>
-<part name="JP1" library="pinhead" deviceset="PINHD-2X3" device="" value="I2C ADDRESS"/>
+<part name="JP2" library="pinhead" deviceset="PINHD-2X3" device="" value="I2C ADDRESS"/>
 <part name="GND10" library="supply1" deviceset="GND" device=""/>
 <part name="P+8" library="SteveMarple" deviceset="AVCC" device=""/>
@@
 <part name="R8" library="SteveMarple" deviceset="RESISTOR" device="1206-HAND" value="3k9"/>
 <part name="R9" library="SteveMarple" deviceset="RESISTOR" device="1206-HAND" value="3k9"/>
-<part name="JP2" library="SparkFun" deviceset="JUMPER-2" device="PTH" value="PROG"/>
+<part name="JP3" library="SparkFun" deviceset="JUMPER-2" device="PTH" value="PROG"/>
 <part name="GND15" library="supply1" deviceset="GND" device=""/>
 <part name="R3" library="SteveMarple" deviceset="RESISTOR" device="1210-HAND" value="4k7"/>
-<part name="JP3" library="SparkFun" deviceset="JUMPER-3" device="PTH" value="I2C VIN"/>
+<part name="JP1" library="SparkFun" deviceset="JUMPER-3" device="PTH" value="I2C VIN"/>
 <part name="U$6" library="SteveMarple" deviceset="PAD" device=""/>
 <part name="U$7" library="SteveMarple" deviceset="PAD" device=""/>
@@
 <instance part="C12" gate="G$1" x="-63.5" y="0"/>
 <instance part="C13" gate="G$1" x="-53.34" y="0"/>
-<instance part="JP1" gate="A" x="40.64" y="-45.72"/>
+<instance part="JP2" gate="A" x="40.64" y="-45.72"/>
 <instance part="GND10" gate="1" x="58.42" y="-60.96"/>
 <instance part="P+8" gate="1" x="58.42" y="-30.48"/>
@@
 <instance part="C1" gate="G$1" x="38.1" y="76.2"/>
 <instance part="R3" gate="G$1" x="83.82" y="73.66" rot="R90"/>
-<instance part="JP3" gate="G$1" x="119.38" y="144.78"/>
+<instance part="JP1" gate="G$1" x="119.38" y="144.78"/>
 <instance part="U$6" gate="G$1" x="177.8" y="48.26"/>
 <instance part="U$7" gate="G$1" x="187.96" y="48.26"/>
@@
 </segment>
 <segment>
-<pinref part="JP1" gate="A" pin="6"/>
+<pinref part="JP2" gate="A" pin="6"/>
 <wire x1="45.72" y1="-48.26" x2="58.42" y2="-48.26" width="0.1524" layer="91"/>
 <pinref part="GND10" gate="1" pin="GND"/>
@@
 <junction x="58.42" y="-55.88"/>
 <wire x1="58.42" y1="-55.88" x2="58.42" y2="-58.42" width="0.1524" layer="91"/>
-<pinref part="JP1" gate="A" pin="5"/>
+<pinref part="JP2" gate="A" pin="5"/>
 <wire x1="38.1" y1="-48.26" x2="33.02" y2="-48.26" width="0.1524" layer="91"/>
 <wire x1="33.02" y1="-48.26" x2="33.02" y2="-55.88" width="0.1524" layer="91"/>
@@
 <label x="106.68" y="142.24" size="1.778" layer="95" rot="MR0"/>
 <wire x1="119.38" y1="139.7" x2="109.22" y2="139.7" width="0.1524" layer="91"/>
-<pinref part="JP3" gate="G$1" pin="1"/>
+<pinref part="JP1" gate="G$1" pin="1"/>
 <wire x1="119.38" y1="142.24" x2="119.38" y2="139.7" width="0.1524" layer="91"/>
 </segment>
@@
 </segment>
 <segment>
-<pinref part="JP1" gate="A" pin="2"/>
+<pinref part="JP2" gate="A" pin="2"/>
 <wire x1="45.72" y1="-43.18" x2="58.42" y2="-43.18" width="0.1524" layer="91"/>
 <pinref part="P+8" gate="1" pin="AVCC"/>
@@
 <junction x="58.42" y="-35.56"/>
 <wire x1="58.42" y1="-35.56" x2="58.42" y2="-33.02" width="0.1524" layer="91"/>
-<pinref part="JP1" gate="A" pin="1"/>
+<pinref part="JP2" gate="A" pin="1"/>
 <wire x1="38.1" y1="-43.18" x2="33.02" y2="-43.18" width="0.1524" layer="91"/>
 <wire x1="33.02" y1="-43.18" x2="33.02" y2="-35.56" width="0.1524" layer="91"/>
@@
 <wire x1="55.88" y1="-12.7" x2="30.48" y2="-12.7" width="0.1524" layer="91"/>
 <wire x1="30.48" y1="-12.7" x2="30.48" y2="-45.72" width="0.1524" layer="91"/>
-<pinref part="JP1" gate="A" pin="3"/>
+<pinref part="JP2" gate="A" pin="3"/>
 <wire x1="30.48" y1="-45.72" x2="38.1" y2="-45.72" width="0.1524" layer="91"/>
 </segment>
@@
 <net name="N$16" class="0">
 <segment>
-<pinref part="JP1" gate="A" pin="4"/>
+<pinref part="JP2" gate="A" pin="4"/>
 <wire x1="45.72" y1="-45.72" x2="53.34" y2="-45.72" width="0.1524" layer="91"/>
 <wire x1="53.34" y1="-45.72" x2="53.34" y2="-15.24" width="0.1524" layer="91"/>
@@
 <wire x1="124.46" y1="88.9" x2="132.08" y2="88.9" width="0.1524" layer="91" style="shortdash"/>
 <junction x="124.46" y="88.9"/>
-<pinref part="JP3" gate="G$1" pin="3"/>
+<pinref part="JP1" gate="G$1" pin="3"/>
 <wire x1="124.46" y1="142.24" x2="124.46" y2="88.9" width="0.1524" layer="91"/>
 </segment>
@@
 <net name="I2C_VIN" class="1">
 <segment>
-<pinref part="JP3" gate="G$1" pin="2"/>
+<pinref part="JP1" gate="G$1" pin="2"/>
 <wire x1="121.92" y1="142.24" x2="121.92" y2="139.7" width="0.1524" layer="91"/>
 <pinref part="X1" gate="G$1" pin="1"/>
@@
 <instance part="R8" gate="G$1" x="233.68" y="147.32" rot="R90"/>
 <instance part="R9" gate="G$1" x="243.84" y="147.32" rot="R90"/>
-<instance part="JP2" gate="A" x="226.06" y="129.54" rot="R270"/>
+<instance part="JP3" gate="A" x="226.06" y="129.54" rot="R270"/>
 <instance part="GND15" gate="1" x="223.52" y="121.92"/>
 </instances>
@@
 </segment>
 <segment>
-<pinref part="JP2" gate="A" pin="2"/>
+<pinref part="JP3" gate="A" pin="2"/>
 <pinref part="GND15" gate="1" pin="GND"/>
 <wire x1="223.52" y1="127" x2="223.52" y2="124.46" width="0.1524" layer="91"/>
@@
 <wire x1="223.52" y1="139.7" x2="215.9" y2="139.7" width="0.1524" layer="91"/>
 <junction x="223.52" y="139.7"/>
-<pinref part="JP2" gate="A" pin="1"/>
+<pinref part="JP3" gate="A" pin="1"/>
 <wire x1="223.52" y1="139.7" x2="223.52" y2="129.54" width="0.1524" layer="91"/>
 </segment>

Commit message: Minor fixes to silkscreen
Other:
- note added: "1 wire interface"
- note added: "ADC"
- note added: "HAT EEPROM"
- note added: "I2C connector, wired for AuroraWatchNet magnetometer sensors but using RJ11"
- note added: "I2C level shifting"
- note added: "Option to not fit a linear regulator"
- note added: "Optional load resistor for DC-DC converter"
- note added: "Raspberry Pi ADC hat"
- note added: "Test pins"
- note removed: "Optional load resistor"
- note removed: "Raspberry Pi Camera Controller"
Changed lines of the file:
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@@
 <wire x1="137.922" y1="115.57" x2="139.192" y2="116.078" width="0.1524" layer="94"/>
 <wire x1="139.192" y1="115.062" x2="137.922" y2="115.57" width="0.1524" layer="94"/>
-<text x="-144.78" y="45.72" size="3.81" layer="91">Raspberry Pi header</text>
-<text x="43.18" y="170.18" size="5.08" layer="91" align="bottom-center">Raspberry Pi Camera Controller</text>
-<text x="101.6" y="53.34" size="2.54" layer="91">AVcc supply</text>
+<text x="43.18" y="170.18" size="5.08" layer="94" align="bottom-center">Raspberry Pi ADC hat</text>
+<text x="101.6" y="53.34" size="3.81" layer="94" ratio="10">AVcc supply</text>
 <text x="48.26" y="88.9" size="1.778" layer="91">Option to not fit a
 DC-DC converter</text>
 <text x="121.92" y="68.58" size="1.778" layer="91">Tantalum</text>
 <text x="172.72" y="68.58" size="1.778" layer="91">Tantalum</text>
-<text x="83.82" y="93.98" size="1.778" layer="91">Optional load
-resistor</text>
+<text x="83.82" y="93.98" size="1.778" layer="91">Optional load resistor
+for DC-DC converter</text>
 <wire x1="88.9" y1="92.71" x2="88.9" y2="77.724" width="0.1524" layer="94"/>
 <wire x1="88.9" y1="77.724" x2="85.09" y2="77.724" width="0.1524" layer="94"/>
@@
 <wire x1="85.09" y1="77.724" x2="87.63" y2="78.486" width="0.1524" layer="94"/>
 <wire x1="87.63" y1="76.962" x2="87.63" y2="78.486" width="0.1524" layer="94"/>
+<text x="-142.24" y="-63.5" size="3.81" layer="94" ratio="10">1 wire interface</text>
+<text x="134.62" y="-30.48" size="3.81" layer="94" ratio="10">I2C level shifting</text>
+<text x="-5.08" y="-58.42" size="3.81" layer="94" ratio="10">ADC</text>
+<text x="-139.7" y="45.72" size="3.81" layer="94" ratio="10">Raspberry Pi header</text>
+<text x="187.96" y="38.1" size="1.778" layer="91">Test pins</text>
+<text x="129.54" y="91.44" size="1.778" layer="91">Option to not fit a
+linear regulator</text>
+<text x="157.48" y="129.54" size="1.778" layer="91">I2C connector, wired for
+AuroraWatchNet magnetometer
+sensors but using RJ11</text>
 </plain>
 <instances>
@@
 <text x="330.962" y="4.318" size="2.54" layer="94">Steve Marple</text>
 <text x="328.422" y="14.478" size="2.54" layer="94">1.0.0</text>
+<text x="205.74" y="101.6" size="3.81" layer="94" ratio="10">HAT EEPROM</text>
 </plain>
 <instances>
